File: ripolab_pcb/ripolab_pcb.sch (KiCad schematic (older format))
At the start: 38 parts, among them J1 Conn_01x02, SW1 SPDT, U1 ESP-12, U2 SPX3819M5-L-3-3

Commit message: badge ripolab v1
Parts:
- added C3: 10nF, Capacitor_SMD:C_0805_2012Metric_Pad1.15x1.50mm_HandSolder, symbol Device:C
- added C4: 47uF, Capacitor_SMD:C_0805_2012Metric_Pad1.15x1.50mm_HandSolder, symbol Device:C
- added D1: D_Schottky_ALT, Diode_SMD:D_SOD-123, symbol Device:D_Schottky_ALT
- added GND_1: GND, ripolab_pcb:TestPad, symbol wickerlib:TEST_1P
- added VCC_1: TEST_VCC, ripolab_pcb:TestPad, symbol wickerlib:TEST_1P
- ADC_1: renamed from ADC1; footprint TestPoint:TestPoint_THTPad_D2.5mm_Drill1.2mm -> ripolab_pcb:TestPad
- C1: value 10nF -> 47uF
- C2: value C -> 100nF
- CH_PD_1: renamed from CH_PD1; footprint TestPoint:TestPoint_THTPad_D2.5mm_Drill1.2mm -> ripolab_pcb:TestPad
- GPIO0: renamed from W7; footprint TestPoint:TestPoint_THTPad_D2.5mm_Drill1.2mm -> ripolab_pcb:TestPad
- GPIO12: renamed from W3; footprint TestPoint:TestPoint_THTPad_D2.5mm_Drill1.2mm -> ripolab_pcb:TestPad
- GPIO13: renamed from W4; footprint TestPoint:TestPoint_THTPad_D2.5mm_Drill1.2mm -> ripolab_pcb:TestPad
- GPIO14: renamed from W2; footprint TestPoint:TestPoint_THTPad_D2.5mm_Drill1.2mm -> ripolab_pcb:TestPad
- GPIO15: renamed from W9; footprint TestPoint:TestPoint_THTPad_D2.5mm_Drill1.2mm -> ripolab_pcb:TestPad
- GPIO16: renamed from W1; footprint TestPoint:TestPoint_THTPad_D2.5mm_Drill1.2mm -> ripolab_pcb:TestPad
- GPIO2: renamed from W8; footprint TestPoint:TestPoint_THTPad_D2.5mm_Drill1.2mm -> ripolab_pcb:TestPad
- GPIO4: renamed from W6; footprint TestPoint:TestPoint_THTPad_D2.5mm_Drill1.2mm -> ripolab_pcb:TestPad
- GPIO5: renamed from W5; footprint TestPoint:TestPoint_THTPad_D2.5mm_Drill1.2mm -> ripolab_pcb:TestPad
- ON1: footprint LEDs:LED_0805_HandSoldering -> LED_SMD:LED_0805_2012Metric
- R7: value R -> 10K
- RST_1: renamed from RESET1; footprint TestPoint:TestPoint_THTPad_D2.5mm_Drill1.2mm -> ripolab_pcb:TestPad
- RX_1: renamed from RX1; footprint TestPoint:TestPoint_THTPad_D2.5mm_Drill1.2mm -> ripolab_pcb:TestPad
- TX_1: renamed from TX1; footprint TestPoint:TestPoint_THTPad_D2.5mm_Drill1.2mm -> ripolab_pcb:TestPad
Connections:
- wire segments 75 -> 84
Other:
- moved on the sheet: C2

Commit message: version 2.0 (corrección v1.0)
Parts:
- removed ADC_1: ADC, ripolab_pcb:TestPad, symbol wickerlib:TEST_1P
- removed CH_PD_1: CH_PD, ripolab_pcb:TestPad, symbol wickerlib:TEST_1P
- removed GPIO0, GPIO12, GPIO13, GPIO14, GPIO15, GPIO16, GPIO2, GPIO4, GPIO5: TEST_1P, ripolab_pcb:TestPad, symbol wickerlib:TEST_1P
- removed U1: ESP-12, ESP8266:ESP-12E_SMD, symbol ESP8266:ESP-12
- added U1: ESP-12E, ESP8266:ESP-12E_SMD, symbol ESP8266:ESP-12E
Connections:
- net labels removed: ADC, GPIO12, GPIO13, GPIO14, GPIO16, GPIO5
- wire segments 84 -> 75
- no-connect marks 3 -> 15
Other:
- moved on the sheet: C1, LED1, LED2, LED3, LED4, LED5, LED6, LED7, LED8
